File: Backup_1.kicad_pcb (KiCad board)
At the start: 2 copper layers, 100 x 100 mm, 75 parts, among them J1 Conn_01x24_ROUND, J2 Conn_01x24_ROUND, J3 Conn_01x31_SQWARE, SW1 SW_Push, SW2 SW_Push, SW3 SW_Push, SW4 SW_Push, U1 PTH04070WAZ, U10 PTH08080W, U2 STM32F378CCTx, U3 PTH04070WAZ, U4 MCP2003, U7 PTN78000HAZ, U8 PTN78000HAZ

Commit message: Last Update 23.04- Verificare butoane/VCC_conn/SWD_conn/Layout
Routing:
- net GND: track 0.00 -> 440.1 mm, vias 0 -> 5
- net +3V3: track 0.00 -> 244.0 mm, vias 0 -> 7
- net +5V: track 0.00 -> 229.3 mm, vias 0 -> 1
- net +15V: track 0.00 -> 165.6 mm
- net SDA2: track 0.00 -> 64.4 mm, vias 0 -> 2
- net SCL2: track 0.00 -> 64.0 mm, vias 0 -> 2
- net (SA0)_Round2: track 0.00 -> 55.8 mm, vias 0 -> 2
- net GPIO_Out_CS1: track 0.00 -> 55.4 mm, vias 0 -> 2
- net WR_Round2: track 0.00 -> 54.6 mm
- net GPIO_Out_CS2: track 0.00 -> 53.5 mm, vias 0 -> 2
- net Net-(D1-Pad4): track 0.00 -> 52.8 mm, vias 0 -> 1
- net SDA1: track 0.00 -> 50.9 mm
- net RES_Round2: track 0.00 -> 49.5 mm
- net SCL1: track 0.00 -> 48.0 mm, vias 0 -> 2
- net RES_Round1: track 0.00 -> 47.6 mm, vias 0 -> 2
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