File: dash-board.kicad_pcb (KiCad board)
At the start: 2 copper layers, 100 x 100 mm, 75 parts, among them J1 Conn_01x24_ROUND, J2 Conn_01x24_ROUND, J3 Conn_01x31_SQWARE, SW1 SW_Push, SW2 SW_Push, SW3 SW_Push, SW4 SW_Push, U1 PTH04070WAZ, U10 PTH08080W, U2 STM32F378CCTx, U3 PTH04070WAZ, U4 MCP2003, U7 PTN78000HAZ, U8 PTN78000HAZ

Commit message: Update 26.04
Layout v2
Parts:
- C1, C2, C3, C4, R1, R2, R3, R4: moved to B.Cu
- SW1, SW2, SW3, SW4: footprint Button_Switch_SMD:SW_SPST_TL3305A -> green-ic-footprint:SW_EVQQ2Y03W
- moved C7 90.4 mm to (127.3, 73.2)
- moved C9 86.9 mm to (126.8, 66.0), turned to 180 degrees
- moved C30 83.1 mm to (63.5, 87.4), turned to 0 degrees
- moved R31 82.4 mm to (127.3, 79.9)
- moved C8 71.5 mm to (116.5, 66.3), turned to 0 degrees
- moved U3 71.0 mm to (118.6, 75.4)
- moved C41 59.4 mm to (63.5, 91.9)
- moved C10 55.7 mm to (90.2, 72.7)
- moved C47 53.3 mm to (70.9, 137.9)
- moved R32 50.1 mm to (65.1, 104.1), turned to 180 degrees
- moved R30 49.3 mm to (89.4, 79.6)
- moved U7 44.6 mm to (65.0, 109.5)
- moved C11 38.8 mm to (71.4, 104.6), turned to 180 degrees
- moved U1 38.7 mm to (81.5, 75.4)
- moved C12 38.6 mm to (77.8, 104.1), turned to 180 degrees
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Routing:
- net GND: track 0.00 -> 261.9 mm, vias 0 -> 8
- net +5V: track 0.00 -> 128.3 mm, vias 0 -> 8
- net +1V8: track 0.00 -> 43.6 mm
- net +12V: track 0.00 -> 37.2 mm
- net Net-(R32-Pad1): track 0.00 -> 24.5 mm
- net +3V3: track 0.00 -> 18.0 mm
- net +24V: track 0.00 -> 13.1 mm
- net +15V: track 0.00 -> 7.40 mm
- net Net-(R31-Pad1): track 0.00 -> 5.79 mm
- net Net-(R30-Pad2): track 0.00 -> 5.13 mm
- net Net-(C35-Pad2): track 0.00 -> 4.92 mm
- net Net-(C33-Pad2): track 0.00 -> 4.38 mm

Commit message: Final Layout
- debug pins
Parts:
- added J4: KLDX-0202-AC, green-ic-footprint:KYCON_KLDX-0202-AC, B.Cu at (53.8, 100.3)
- moved C41 51.4 mm to (114.8, 95.3), turned to 270 degrees
- moved U4 45.5 mm to (121.7, 95.0), turned to 0 degrees
- moved C47 40.2 mm to (66.0, 98.0), turned to 90 degrees
- moved C28 7.24 mm to (124.7, 63.5), turned to 0 degrees
- moved C26 7.12 mm to (104.6, 63.5), turned to 0 degrees
- moved C20 7.12 mm to (75.5, 63.5), turned to 0 degrees
- moved C21 7.11 mm to (85.6, 63.5), turned to 0 degrees
- moved C25 7.11 mm to (94.7, 63.5), turned to 0 degrees
- moved C27 7.11 mm to (115.1, 63.5), turned to 0 degrees
- moved C19 7.11 mm to (65.7, 65.3), turned to 0 degrees
- moved C29 6.99 mm to (135.1, 65.3), turned to 0 degrees
- moved C9 6.26 mm to (121.6, 69.6)
- moved C6 6.20 mm to (84.5, 69.6)
- moved C43 5.59 mm to (63.5, 84.3)
- moved C32 5.59 mm to (136.4, 77.7)
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Connections:
- net MISO renamed SWJ-DP
- net Net-(U2-Pad7) renamed NRST
Routing:
- net +3V3: track 18.0 -> 270.6 mm, vias 0 -> 11
- net +15V: track 7.40 -> 256.8 mm, vias 0 -> 8
- net Net-(R1-Pad2): track 0.00 -> 145.3 mm, vias 0 -> 4
- net GND: track 261.9 -> 121.7 mm, vias 8 -> 25
- net Net-(C4-Pad1): track 0.00 -> 121.9 mm, vias 0 -> 4
- net +12V: track 37.2 -> 147.5 mm, vias 0 -> 4
- net Net-(C3-Pad1): track 0.00 -> 99.1 mm, vias 0 -> 3
- net +24V: track 13.1 -> 101.6 mm
- net Net-(C2-Pad1): track 0.00 -> 86.8 mm, vias 0 -> 3
- net +5V: track 128.3 -> 214.0 mm, vias 8 -> 10
- net WR_Round2: track 0.00 -> 75.6 mm, vias 0 -> 4
- net Net-(D1-Pad4): track 0.00 -> 72.0 mm, vias 0 -> 1
- net SDA1: track 0.00 -> 68.5 mm, vias 0 -> 4
- net Net-(C1-Pad1): track 0.00 -> 67.7 mm, vias 0 -> 3
- net SCL1: track 0.00 -> 65.5 mm, vias 0 -> 4
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Other:
- rule trace_min: 0.2 -> 0
- rule via_min_size: 0.4 -> 0.1

Commit message: layout changes
Parts:
- added J5: Conn_01x04_Male, Connector_PinHeader_2.54mm:PinHeader_1x04_P2.54mm_Vertical, F.Cu at (146.0, 94.3)
- moved R35 19.5 mm to (110.5, 123.3), turned to 90 degrees
- moved C6 6.47 mm to (88.9, 74.4), turned to 270 degrees
- moved C15 3.09 mm to (124.2, 104.7), turned to 270 degrees
- moved C10 2.54 mm to (92.7, 75.4)
- moved C20 2.10 mm to (74.0, 65.0), turned to 270 degrees
- moved C19 2.03 mm to (64.3, 66.7), turned to 270 degrees
- moved C11 1.95 mm to (73.0, 105.8), turned to 0 degrees
- moved C27 1.91 mm to (113.6, 64.7), turned to 270 degrees
- moved C25 1.89 mm to (93.1, 64.5), turned to 270 degrees
- moved C29 1.82 mm to (133.7, 66.4), turned to 270 degrees
- moved C26 1.81 mm to (103.1, 64.5), turned to 270 degrees
- moved C28 1.73 mm to (123.2, 64.4), turned to 270 degrees
- moved C21 1.69 mm to (84.2, 64.5), turned to 270 degrees
- moved C22 1.51 mm to (91.2, 109.8), turned to 90 degrees
- moved C5 0.98 mm to (79.5, 69.6)
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Connections:
- U2 pad 34: SWJ-DP -> MISO
Routing:
- net MISO: track 0.00 -> 44.2 mm
- net +5V: track 214.0 -> 184.8 mm
- net SWJ-DP: track 29.0 -> 0.00 mm, vias 3 -> 0
- net +12V: track 147.5 -> 128.4 mm
- net NRST: track 38.3 -> 56.7 mm, vias 3 -> 2
- net +24V: track 101.6 -> 86.7 mm
- net Net-(R35-Pad1): track 18.2 -> 3.82 mm
- net GND: track 121.7 -> 111.7 mm, vias 25 -> 21
- net +1V8: track 57.8 -> 53.3 mm
- net Net-(C4-Pad1): track 121.9 -> 120.1 mm
- net +3V3: track 270.6 -> 272.1 mm
- net +15V: track 256.8 -> 258.1 mm

Commit message: layout final 2.0
Routing:
- net GND: track 111.7 -> 79.0 mm, vias 21 -> 22
Changed lines of the file:
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@@
-(kicad_pcb (version 20171130) (host pcbnew "(5.1.5)-3")
+(kicad_pcb (version 20171130) (host pcbnew "(5.1.0)-1")
   (general
     (thickness 1.6)
     (drawings 149)
-    (tracks 840)
+    (tracks 828)
     (zones 0)
     (modules 77)
@@
   (segment (start 142.506 86.856) (end 143.002 86.36) (width 0.25) (layer B.Cu) (net 1))
   (segment (start 140.925 86.856) (end 142.506 86.856) (width 0.25) (layer B.Cu) (net 1))
-  (via (at 81.4 106) (size 0.8) (drill 0.4) (layers F.Cu B.Cu) (net 1))
-  (segment (start 58.2 68.292) (end 56.896 69.596) (width 0.25) (layer F.Cu) (net 1))
-  (segment (start 67.31 55.63) (end 66.484999 54.804999) (width 0.25) (layer F.Cu) (net 1))
-  (segment (start 58.2 57.1) (end 58.2 68.292) (width 0.25) (layer F.Cu) (net 1))
-  (segment (start 67.31 55.88) (end 67.31 55.63) (width 0.25) (layer F.Cu) (net 1))
-  (segment (start 66.484999 54.804999) (end 60.495001 54.804999) (width 0.25) (layer F.Cu) (net 1))
-  (segment (start 60.495001 54.804999) (end 58.2 57.1) (width 0.25) (layer F.Cu) (net 1))
-  (segment (start 104.14 89.408) (end 102.592 89.408) (width 0.25) (layer B.Cu) (net 1))
-  (segment (start 102.326 89.674) (end 102.326 90.8335) (width 0.25) (layer B.Cu) (net 1))
-  (segment (start 102.592 89.408) (end 102.326 89.674) (width 0.25) (layer B.Cu) (net 1))
-  (segment (start 123.571 95.885) (end 123.571 97.696) (width 0.25) (layer B.Cu) (net 1))
-  (segment (start 122.9 95.2) (end 123.571 95.885) (width 0.25) (layer B.Cu) (net 1))
-  (segment (start 122.301 94.601) (end 122.9 95.2) (width 0.25) (layer B.Cu) (net 1))
-  (segment (start 122.301 92.296) (end 122.301 94.601) (width 0.25) (layer B.Cu) (net 1))
+  (via (at 131.572 100.457) (size 0.8) (drill 0.4) (layers F.Cu B.Cu) (net 1))
+  (via (at 136.017 77.47) (size 0.8) (drill 0.4) (layers F.Cu B.Cu) (net 1))
   (segment (start 99.51621 107.97121) (end 98.733 107.188) (width 0.919283) (layer B.Cu) (net 2))
   (segment (start 102.407357 110.862357) (end 99.51621 107.97121) (width 0.919283) (layer B.Cu) (net 2))
@@
   (segment (start 140.007364 77.724) (end 139.7 77.724) (width 0.25) (layer B.Cu) (net 32))
   (segment (start 139.7 77.724) (end 139.503002 77.724) (width 0.25) (layer B.Cu) (net 32))
-  (via (at 133.313 79.091) (size 0.8) (drill 0.4) (layers F.Cu B.Cu) (net 32))
-  (segment (start 133.34901 79.05499) (end 133.313 79.091) (width 0.25) (layer B.Cu) (net 32))
-  (segment (start 133.34901 76.07399) (end 133.34901 79.05499) (width 0.25) (layer B.Cu) (net 32))
   (segment (start 133.34901 76.07399) (end 136.27199 76.07399) (width 0.25) (layer B.Cu) (net 32))
   (segment (start 130.70399 76.07399) (end 133.34901 76.07399) (width 0.25) (layer B.Cu) (net 32))
@@
   (segment (start 146 94.3) (end 143.6 94.3) (width 0.25) (layer B.Cu) (net 32))
   (segment (start 143.6 94.3) (end 141.9 96) (width 0.25) (layer B.Cu) (net 32))
+  (segment (start 133.34901 79.05499) (end 133.313 79.091) (width 0.25) (layer B.Cu) (net 32))
+  (segment (start 133.34901 76.07399) (end 133.34901 79.05499) (width 0.25) (layer B.Cu) (net 32))
+  (via (at 133.313 79.091) (size 0.8) (drill 0.4) (layers F.Cu B.Cu) (net 32))
   (segment (start 140.925 80.856) (end 136.99 80.856) (width 0.25) (layer B.Cu) (net 33))
   (segment (start 101.826 90.8335) (end 101.826 88.928) (width 0.25) (layer B.Cu) (net 33))
@@
   (segment (start 132.588 81.534) (end 136.77799 81.534) (width 0.25) (layer B.Cu) (net 47))
   (via (at 132.588 77.47) (size 0.8) (drill 0.4) (layers F.Cu B.Cu) (net 47))
-  (segment (start 132.588 77.47) (end 132.588 81.534) (width 0.25) (layer F.Cu) (net 47))
-  (segment (start 131.064 77.47) (end 132.588 77.47) (width 0.25) (layer B.Cu) (net 47))
-  (segment (start 130.81 77.47) (end 131.064 77.47) (width 0.25) (layer B.Cu) (net 47))
+  (segment (start 91.948 79.756) (end 128.524 79.756) (width 0.25) (layer B.Cu) (net 47))
   (segment (start 128.524 79.756) (end 130.81 77.47) (width 0.25) (layer B.Cu) (net 47))
+  (segment (start 130.81 77.47) (end 131.064 77.47) (width 0.25) (layer B.Cu) (net 47))
+  (segment (start 131.064 77.47) (end 132.588 77.47) (width 0.25) (layer B.Cu) (net 47))
+  (segment (start 132.588 77.47) (end 132.588 81.534) (width 0.25) (layer F.Cu) (net 47))
   (segment (start 91.44 80.264) (end 91.948 79.756) (width 0.25) (layer B.Cu) (net 47))
-  (segment (start 91.948 79.756) (end 128.524 79.756) (width 0.25) (layer B.Cu) (net 47))
   (via (at 71.118075 81.282581) (size 0.8) (drill 0.4) (layers F.Cu B.Cu) (net 48))
   (segment (start 58.846 80.776) (end 70.611494 80.776) (width 0.25) (layer B.Cu) (net 48))
@@
   (segment (start 106.174 96.774) (end 106.172 96.774) (width 0.25) (layer B.Cu) (net 84))
   (segment (start 108.46 99.06) (end 106.174 96.774) (width 0.25) (layer B.Cu) (net 84))
-  (segment (start 104.2385 96.746) (end 105.201596 96.746) (width 0.25) (layer B.Cu) (net 86))
-  (segment (start 105.201596 96.746) (end 105.902742 97.447146) (width 0.25) (layer B.Cu) (net 86))
   (via (at 101.854 95.885) (size 0.8) (drill 0.4) (layers F.Cu B.Cu) (net 85))
   (segment (start 95.9135 94.746) (end 100.715 94.746) (width 0.25) (layer B.Cu) (net 85))
@@
   (segment (start 104.394 100.457) (end 129.643 100.457) (width 0.25) (layer B.Cu) (net 85))
   (segment (start 129.643 100.457) (end 132.6 97.5) (width 0.25) (layer B.Cu) (net 85))
+  (segment (start 104.2385 96.746) (end 105.201596 96.746) (width 0.25) (layer B.Cu) (net 86))
+  (segment (start 105.201596 96.746) (end 105.902742 97.447146) (width 0.25) (layer B.Cu) (net 86))
   (segment (start 129.1 99.7) (end 128.985001 99.785001) (width 0.25) (layer B.Cu) (net 86))
   (segment (start 131.96 96.84) (end 129.1 99.7) (width 0.25) (layer B.Cu) (net 86))
